Commit message: fk-intrin: added eval script, fixed joint limits in iiwa urdf

File: models/iiwa/iiwa_rbd_accel.urdf (robot description, URDF)
Before this commit: robot iiwa, 8 links, 7 joints
Joints:
- joint lbr_iiwa_joint_1: limit lower=-100000.0 upper=100000.0 effort=30.0 velocity=1.0 -> lower=-2.9671 upper=2.9671 effort=30.0 velocity=1.0
- joint lbr_iiwa_joint_2: limit lower=-100000.0 upper=100000.0 effort=30.0 velocity=1.0 -> lower=-2.0944 upper=2.0944 effort=30.0 velocity=1.0
- joint lbr_iiwa_joint_3: limit lower=-100000.0 upper=100000.0 effort=30.0 velocity=1.0 -> lower=-2.9671 upper=2.9671 effort=30.0 velocity=1.0
- joint lbr_iiwa_joint_4: limit lower=-100000.0 upper=100000.0 effort=30.0 velocity=1.0 -> lower=-2.0944 upper=2.0944 effort=30.0 velocity=1.0
- joint lbr_iiwa_joint_5: limit lower=-100000.0 upper=100000.0 effort=30.0 velocity=1.0 -> lower=-2.9671 upper=2.9671 effort=30.0 velocity=1.0
- joint lbr_iiwa_joint_6: limit lower=-100000.0 upper=100000.0 effort=30.0 velocity=1.0 -> lower=-2.0944 upper=2.0944 effort=30.0 velocity=1.0
- joint lbr_iiwa_joint_7: limit lower=-100000.0 upper=100000.0 effort=30.0 velocity=1.0 -> lower=-3.0543 upper=3.0543 effort=30.0 velocity=1.0
